File: AR488-esp32-devkitc/AR488-esp32-devkitc.kicad_pcb (KiCad board)
At the start: 2 copper layers, 63.5 x 50 mm, 7 parts, among them J2 Conn_02x12_Odd_Even, U2 ESP32-DevKitC

Commit message: Sent to board fab
No version markings. 5x of each:
- Common
- Common-nobuffer
- ESP32-devkitc
- ESP32-S3-devkitc
Parts:
- added REF**: Order_Label, JLCPCB_tools:Order_Label, B.Cu at (123.2, 107.3)
