File: AR488-esp32-devkitc/AR488-esp32-devkitc.kicad_sch (KiCad schematic)
At the start: 2 parts

Commit message: Sent to board fab
No version markings. 5x of each:
- Common
- Common-nobuffer
- ESP32-devkitc
- ESP32-S3-devkitc
Parts:
- J2: value (none) -> Conn_02x12_Odd_Even; footprint (none) -> Connector_PinHeader_2.54mm:PinHeader_2x12_P2.54mm_Vertical
- U2: value (none) -> ESP32-DevKitC; footprint (none) -> esp32:ESP32-DevKitC
Changed lines of the file:
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@@
     (in_bom yes) (on_board yes)
     (property "Reference" "J2" (id 0) (at 94.615 37.0332 0))
-    (property "Value" "" (id 1) (at 94.615 39.3446 0))
-    (property "Footprint" "" (id 2) (at 93.345 55.245 0)
+    (property "Value" "Conn_02x12_Odd_Even" (id 1) (at 94.615 39.3446 0))
+    (property "Footprint" "Connector_PinHeader_2.54mm:PinHeader_2x12_P2.54mm_Vertical" (id 2) (at 93.345 55.245 0)
       (effects (font (size 1.27 1.27)) hide)
     )
@@
       (effects (font (size 1.27 1.27)) hide)
     )
-    (property "Value" "" (id 1) (at 124.5108 84.074 0))
+    (property "Value" "+5V" (id 1) (at 124.5108 84.074 0))
     (property "Footprint" "" (id 2) (at 128.905 84.455 0)
       (effects (font (size 1.27 1.27)) hide)
@@
       (effects (font (size 1.27 1.27)) hide)
     )
-    (property "Value" "" (id 1) (at 106.045 55.245 90))
+    (property "Value" "GND" (id 1) (at 106.045 55.245 90))
     (property "Footprint" "" (id 2) (at 100.965 55.245 0)
       (effects (font (size 1.27 1.27)) hide)
@@
       (effects (font (size 1.27 1.27)) hide)
     )
-    (property "Value" "" (id 1) (at 83.185 55.245 90))
+    (property "Value" "GND" (id 1) (at 83.185 55.245 90))
     (property "Footprint" "" (id 2) (at 88.265 55.245 0)
       (effects (font (size 1.27 1.27)) hide)
@@
       (effects (font (size 1.27 1.27)) hide)
     )
-    (property "Value" "" (id 1) (at 105.41 52.705 90))
+    (property "Value" "+5V" (id 1) (at 105.41 52.705 90))
     (property "Footprint" "" (id 2) (at 100.965 52.705 0)
       (effects (font (size 1.27 1.27)) hide)
@@
       (effects (font (size 1.27 1.27)) hide)
     )
-    (property "Value" "" (id 1) (at 83.185 52.705 90))
+    (property "Value" "+5V" (id 1) (at 83.185 52.705 90))
     (property "Footprint" "" (id 2) (at 88.265 52.705 0)
       (effects (font (size 1.27 1.27)) hide)
@@
       (effects (font (size 1.27 1.27)) hide)
     )
-    (property "Value" "" (id 1) (at 83.185 70.485 90))
+    (property "Value" "GND" (id 1) (at 83.185 70.485 90))
     (property "Footprint" "" (id 2) (at 88.265 70.485 0)
       (effects (font (size 1.27 1.27)) hide)
@@
     (in_bom yes) (on_board yes)
     (property "Reference" "U2" (id 0) (at 163.83 30.734 0))
-    (property "Value" "" (id 1) (at 163.83 33.0454 0))
-    (property "Footprint" "" (id 2) (at 161.925 92.075 0)
+    (property "Value" "ESP32-DevKitC" (id 1) (at 163.83 33.0454 0))
+    (property "Footprint" "esp32:ESP32-DevKitC" (id 2) (at 161.925 92.075 0)
       (effects (font (size 1.27 1.27)) hide)
     )
@@
       (effects (font (size 1.27 1.27)) hide)
     )
-    (property "Value" "" (id 1) (at 203.1492 38.608 0))
+    (property "Value" "GND" (id 1) (at 203.1492 38.608 0))
     (property "Footprint" "" (id 2) (at 198.755 38.735 0)
       (effects (font (size 1.27 1.27)) hide)
@@
       (effects (font (size 1.27 1.27)) hide)
     )
-    (property "Value" "" (id 1) (at 124.5108 71.882 0))
+    (property "Value" "GND" (id 1) (at 124.5108 71.882 0))
     (property "Footprint" "" (id 2) (at 128.905 71.755 0)
       (effects (font (size 1.27 1.27)) hide)
@@
       (effects (font (size 1.27 1.27)) hide)
     )
-    (property "Value" "" (id 1) (at 203.1492 53.848 0))
+    (property "Value" "GND" (id 1) (at 203.1492 53.848 0))
     (property "Footprint" "" (id 2) (at 198.755 53.975 0)
       (effects (font (size 1.27 1.27)) hide)
